Commit message: some patches

File: src/spiderproj_description/urdf/spiderproj.xacro (robot description, xacro)
@@ -52,5 +52,5 @@
   <xacro:property name="body_ixx" value="0.00329495565" />
   <xacro:property name="body_iyy" value="0.00422550506" />
-  <xacro:property name="body_izz" value="0.00610423987" />9254901960784314
+  <xacro:property name="body_izz" value="0.00610423987" />
   <xacro:property name="body_ixy" value="-0.00000818428" />
   <xacro:property name="body_ixz" value="-0.00007183633" />
@@ -121,5 +121,5 @@
   <xacro:property name="tibia_R_roll" value="0" />
   <xacro:property name="tibia_R_pitch" value="0" />
-  <xacro:property name="tibia_R_yaw" value="0" />install ros2 hunble
+  <xacro:property name="tibia_R_yaw" value="0" />
   <xacro:property name="tibia_R_ixx" value="0.00004499197" />
   <xacro:property name="tibia_R_iyy" value="0.00019412525" />

Commit message: easier to launch rviz2

File: src/spiderproj_description/urdf/spiderproj.xacro (robot description, xacro)
@@ -190,6 +190,5 @@
       <origin xyz="0 0 0.007" rpy="0 0 ${pi/2}" />
       <geometry>
-        <mesh filename="file://$(find spiderproj_description)/meshes/visual/Body6.stl"
-          scale="1 1 1" />
+        <mesh filename="file://$(find spiderproj_description)/meshes/Body6.stl" scale="1 1 1" />
       </geometry>
       <material name="white_pla" />
@@ -241,5 +240,5 @@
         <origin xyz="0 0 0" rpy="${pi} 0 ${pi}" />
         <geometry>
-          <mesh filename="file://$(find spiderproj_description)/meshes/visual/Coxa_${side}.stl"
+          <mesh filename="file://$(find spiderproj_description)/meshes/Coxa_${side}.stl"
             scale="1 1 1" />
         </geometry>
@@ -285,5 +284,5 @@
         <origin xyz="0 0 -0.0018" rpy="-${pi/2} 0 0" />
         <geometry>
-          <mesh filename="file://$(find spiderproj_description)/meshes/visual/Femur_${side}.stl"
+          <mesh filename="file://$(find spiderproj_description)/meshes/Femur_${side}.stl"
             scale="1 1 1" />
         </geometry>
@@ -337,5 +336,5 @@
         <origin xyz="0 0 0" rpy="-${pi/2} 0 ${pi/2}" />
         <geometry>
-          <mesh filename="file://$(find spiderproj_description)/meshes/visual/Tibia_${side}.stl"
+          <mesh filename="file://$(find spiderproj_description)/meshes/Tibia_${side}.stl"
             scale="1 1 1" />
         </geometry>
